Commit message: Working Sim and Nav stack. No mjaors needed.

File: src/turtlebot3_simulations/turtlebot3_gazebo/urdf/turtlebot3_enemy_bot.urdf (robot description, URDF)
Before this commit: robot turtlebot3_burger_cam, 10 links, 9 joints
Links:
- removed link base_footprint
- removed link base_link
- removed link base_scan
- removed link camera_link
- removed link camera_rgb_frame
- removed link camera_rgb_optical_frame
- removed link caster_back_link
- removed link imu_link
- removed link wheel_left_link
- removed link wheel_right_link
- added link enemy_bot/base_footprint
- added link enemy_bot/base_link, mass 8.2573504e-01; collision box size=0.140 0.140 0.143; visual mesh filename=package://turtlebot3_gazebo/models/turtlebot3_common/meshes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 scale=0.001 0.001 0.001
- added link enemy_bot/base_scan, mass 0.114; collision cylinder length=0.0315 radius=0.055; visual mesh filename=package://turtlebot3_gazebo/models/turtlebot3_common/meshes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 scale=0.001 0.001 0.001
- added link enemy_bot/camera_link; collision box size=0.015 0.030 0.027
- added link enemy_bot/camera_rgb_frame
- added link enemy_bot/camera_rgb_optical_frame
- added link enemy_bot/caster_back_link, mass 0.005; collision box size=0.030 0.009 0.020
- added link enemy_bot/imu_link
- added link enemy_bot/wheel_left_link, mass 2.8498940e-02; collision cylinder length=0.018 radius=0.033; visual mesh filename=package://turtlebot3_gazebo/models/turtlebot3_common/meshes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 scale=0.001 0.001 0.001
- added link enemy_bot/wheel_right_link, mass 2.8498940e-02; collision cylinder length=0.018 radius=0.033; visual mesh filename=package://turtlebot3_gazebo/models/turtlebot3_common/meshes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 scale=0.001 0.001 0.001
Joints:
- joint base_joint: child base_link -> enemy_bot/base_link; parent base_footprint -> enemy_bot/base_footprint
- joint camera_joint: child camera_link -> enemy_bot/camera_link; parent base_link -> enemy_bot/base_link
- joint camera_rgb_joint: child camera_rgb_frame -> enemy_bot/camera_rgb_frame; parent camera_link -> enemy_bot/camera_link
- joint camera_rgb_optical_joint: child camera_rgb_optical_frame -> enemy_bot/camera_rgb_optical_frame; parent camera_rgb_frame -> enemy_bot/camera_rgb_frame
- joint caster_back_joint: child caster_back_link -> enemy_bot/caster_back_link; parent base_link -> enemy_bot/base_link
- joint imu_joint: child imu_link -> enemy_bot/imu_link; parent base_link -> enemy_bot/base_link
- joint scan_joint: child base_scan -> enemy_bot/base_scan; parent base_link -> enemy_bot/base_link
- joint wheel_left_joint: child wheel_left_link -> enemy_bot/wheel_left_link; parent base_link -> enemy_bot/base_link
- joint wheel_right_joint: child wheel_right_link -> enemy_bot/wheel_right_link; parent base_link -> enemy_bot/base_link

File: src/turtlebot3_simulations/turtlebot3_gazebo/urdf/turtlebot3_our_bot.urdf (robot description, URDF)
Before this commit: robot turtlebot3_burger_cam, 10 links, 9 joints
Links:
- removed link base_footprint
- removed link base_link
- removed link base_scan
- removed link camera_link
- removed link camera_rgb_frame
- removed link camera_rgb_optical_frame
- removed link caster_back_link
- removed link imu_link
- removed link wheel_left_link
- removed link wheel_right_link
- added link our_bot/base_footprint
- added link our_bot/base_link, mass 8.2573504e-01; collision box size=0.140 0.140 0.143; visual mesh filename=package://turtlebot3_gazebo/models/turtlebot3_common/meshes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 scale=0.001 0.001 0.001
- added link our_bot/base_scan, mass 0.114; collision cylinder length=0.0315 radius=0.055; visual mesh filename=package://turtlebot3_gazebo/models/turtlebot3_common/meshes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 scale=0.001 0.001 0.001
- added link our_bot/camera_link; collision box size=0.015 0.030 0.027
- added link our_bot/camera_rgb_frame
- added link our_bot/camera_rgb_optical_frame
- added link our_bot/caster_back_link, mass 0.005; collision box size=0.030 0.009 0.020
- added link our_bot/imu_link
- added link our_bot/wheel_left_link, mass 2.8498940e-02; collision cylinder length=0.018 radius=0.033; visual mesh filename=package://turtlebot3_gazebo/models/turtlebot3_common/meshes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 scale=0.001 0.001 0.001
- added link our_bot/wheel_right_link, mass 2.8498940e-02; collision cylinder length=0.018 radius=0.033; visual mesh filename=package://turtlebot3_gazebo/models/turtlebot3_common/meshes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 scale=0.001 0.001 0.001
Joints:
- joint base_joint: child base_link -> our_bot/base_link; parent base_footprint -> our_bot/base_footprint
- joint camera_joint: child camera_link -> our_bot/camera_link; parent base_link -> our_bot/base_link
- joint camera_rgb_joint: child camera_rgb_frame -> our_bot/camera_rgb_frame; parent camera_link -> our_bot/camera_link
- joint camera_rgb_optical_joint: child camera_rgb_optical_frame -> our_bot/camera_rgb_optical_frame; parent camera_rgb_frame -> our_bot/camera_rgb_frame
- joint caster_back_joint: child caster_back_link -> our_bot/caster_back_link; parent base_link -> our_bot/base_link
- joint imu_joint: child imu_link -> our_bot/imu_link; parent base_link -> our_bot/base_link
- joint scan_joint: child base_scan -> our_bot/base_scan; parent base_link -> our_bot/base_link
- joint wheel_left_joint: child wheel_left_link -> our_bot/wheel_left_link; parent base_link -> our_bot/base_link
- joint wheel_right_joint: child wheel_right_link -> our_bot/wheel_right_link; parent base_link -> our_bot/base_link
